Commit message: added more comparisions after submission of rebuttal paper

File: calibrated_urdf/fr3/panda.urdf (robot description, URDF)
Before this commit: robot panda, 14 links, 13 joints
Joints:
- joint ball_joint: origin xyz=-0.0009570680790377462 -0.007030862633004773 0.03339974344028835 rpy=0.0 0.0 0.0 -> xyz=-0.0009679561602663274 -0.007119983214043715 0.03289641687705243 rpy=0.0 0.0 0.0
- joint panda_joint1: origin xyz=-5.5331096994303595e-19 5.483098518124614e-19 0.333 rpy=-3.881509365452199e-18 8.521282659020046e-18 -2.818384959880011e-18 -> xyz=4.049751722273528e-18 6.249934431302164e-18 0.333 rpy=2.3891596660642845e-18 -4.558962715469791e-18 1.183214981704776e-18
- joint panda_joint2: origin xyz=-0.00016195193782980375 0.0003584627092071496 1.5175290806929636e-18 rpy=-1.5692176608432886 -0.0006232911183152322 1.7864692191458248e-08 -> xyz=0.00015992930620912919 0.00016537995304946915 -1.612625971446023e-19 rpy=-1.5688193853667922 0.0005439852849545671 9.75778867075954e-10
- joint panda_joint3: origin xyz=-2.020465809259206e-05 -0.31638865532398874 0.0003584575138760347 rpy=1.5692123307818817 0.006679319093088354 -0.0006168233947439105 -> xyz=-3.631045205078406e-05 -0.316697140343035 0.00016538044311063861 rpy=1.5698897856808722 -0.0022277143821921017 0.0005554730833655623
- joint panda_joint4: origin xyz=0.08205066859185202 -0.0009976171770812098 0.00038937663180532424 rpy=1.5721524306760986 0.00046446560970461926 -0.006597971336104339 -> xyz=0.0822744429253914 0.0004274025276758699 0.0006972686818953394 rpy=1.5692385242654587 0.0008967847005295781 0.0021929508660798376
- joint panda_joint5: origin xyz=-0.08274276254819034 0.3843792920170425 0.0010001543411157804 rpy=-1.5694466120909343 0.00348120156019702 -0.0005176948450394379 -> xyz=-0.08209909546126871 0.3847751240945391 -0.0004268082018264021 rpy=-1.5720416242662738 0.009112100934962829 -0.0006754803382516836
- joint panda_joint6: origin xyz=-0.00012809341151093876 0.0006114705144863913 0.00038038616638708453 rpy=1.5678903763020455 0.0008804283250090152 0.0034804960271833806 -> xyz=0.0008149146228504592 0.0011270403110451585 0.0007759213813046541 rpy=1.5707145079824067 0.0004267431405131075 0.009112918466830345
- joint panda_joint7: origin xyz=0.08519872598122621 4.308755776248788e-06 -0.0006108393557751972 rpy=1.5709914845994533 5.0372969287365315e-08 -0.0008706911908268 -> xyz=0.087001581888464 2.2984836531718647e-06 -0.0011195581933036909 rpy=1.5710591503330307 1.5080950164913995e-07 -0.00042619955982247103

File: calibrated_urdf/panda_2/panda.urdf (robot description, URDF)
Before this commit: robot panda, 14 links, 13 joints
Joints:
- joint ball_joint: origin xyz=0.00037990524928465026 -4.420572608777121e-05 0.03102464075322382 rpy=0.0 0.0 0.0 -> xyz=0.0003752049809680507 0.00018606599493192026 0.03200584380492406 rpy=0.0 0.0 0.0
- joint panda_joint1: origin xyz=-1.2758753865242616e-16 -5.2222054042510136e-17 0.333 rpy=8.366805516041043e-06 8.814350308898128e-08 2.4513630387076608e-17 -> xyz=-3.719447892371078e-19 -8.163891922061419e-19 0.333 rpy=-2.133072628858994e-18 6.549249448272412e-20 2.493742150121163e-19
- joint panda_joint2: origin xyz=-0.00019417564815309772 -0.00018772077543271004 1.796911857934499e-17 rpy=-1.5725347107345484 0.0009255042963167639 -2.2321032908662564e-15 -> xyz=-0.00028650233048617825 0.00013056502818906737 2.7194336891652045e-18 rpy=-1.569248140739377 0.00026947630631280297 -3.0809028052379674e-10
- joint panda_joint3: origin xyz=0.0003371033096498455 -0.31626505724737547 -0.0001877201793910496 rpy=1.5720487481374692 0.00011271550591184526 0.0008189810488676046 -> xyz=0.0002692541027170446 -0.3159009901596097 0.00013056472297234668 rpy=1.5699604016308881 0.0003109596136488854 0.00018439181487172126
- joint panda_joint4: origin xyz=0.08250428687456778 -0.0002847200612681194 0.0002655680887159182 rpy=1.5741434757926136 0.011776708120902118 -9.025189862699405e-05 -> xyz=0.08208705071931605 5.166335696027022e-06 -9.885030163165646e-05 rpy=1.570376081759264 0.0034388237877875996 -0.00031122798628267366
- joint panda_joint5: origin xyz=-0.07866941844576122 0.38493907517903264 0.000283829074942361 rpy=-1.569359416779495 0.005129171736623614 -0.01022805489571219 -> xyz=-0.0816182275577414 0.3841662158400614 -5.0821853736684e-06 rpy=-1.5707024933627616 0.0012570554762050068 -0.003086645893116907
- joint panda_joint6: origin xyz=0.0006537446895798644 -1.275492785867517e-05 0.0009786397273711831 rpy=1.5705258868617893 -0.00043533480446275005 0.005114480048959338 -> xyz=-2.0759871214702803e-05 0.0005000261141171843 0.00016895723105205126 rpy=1.5685773976315296 7.670870280695487e-05 0.0012567567700178502
- joint panda_joint7: origin xyz=0.0902493646325364 -0.0008951821978016663 1.636289653042385e-05 rpy=1.5707208785930096 2.6320186308338895e-08 0.0005154940135814471 -> xyz=0.0876934564010052 1.7029351416458937e-06 -0.0004996729263786812 rpy=1.570917724680222 1.5345168143402714e-08 -7.404089563013065e-05

File: calibrated_urdf/panda_2_bis/panda.urdf (robot description, URDF)
Before this commit: robot panda, 14 links, 13 joints
Joints:
- joint ball_joint: origin xyz=-0.0009570680790377462 -0.007030862633004773 0.03339974344028835 rpy=0.0 0.0 0.0 -> xyz=0.00020330354395513736 -0.0001642671713580531 0.03262822761207553 rpy=0.0 0.0 0.0
- joint panda_joint1: origin xyz=-5.5331096994303595e-19 5.483098518124614e-19 0.333 rpy=-3.881509365452199e-18 8.521282659020046e-18 -2.818384959880011e-18 -> xyz=4.6180249515592785e-17 -4.4404365996626007e-17 0.333 rpy=-1.342677435023694e-17 2.1398695986746344e-17 -1.816623198688617e-17
- joint panda_joint2: origin xyz=-0.00016195193782980375 0.0003584627092071496 1.5175290806929636e-18 rpy=-1.5692176608432886 -0.0006232911183152322 1.7864692191458248e-08 -> xyz=7.492551483196854e-05 0.00014662053139369863 -2.151503663494446e-17 rpy=-1.5694069411837093 0.0004157262981544786 -1.5176844907533936e-06
- joint panda_joint3: origin xyz=-2.020465809259206e-05 -0.31638865532398874 0.0003584575138760347 rpy=1.5692123307818817 0.006679319093088354 -0.0006168233947439105 -> xyz=1.0593988688794304e-05 -0.3163377911725477 0.00014610527035570622 rpy=1.5699239268203637 0.00023702152639266835 0.0004127288729814325
- joint panda_joint4: origin xyz=0.08205066859185202 -0.0009976171770812098 0.00038937663180532424 rpy=1.5721524306760986 0.00046446560970461926 -0.006597971336104339 -> xyz=0.0824800866674542 -4.111896586669298e-06 0.00033665079636207803 rpy=1.5703758251339501 0.003645543458361813 -0.0002352845370055769
- joint panda_joint5: origin xyz=-0.08274276254819034 0.3843792920170425 0.0010001543411157804 rpy=-1.5694466120909343 0.00348120156019702 -0.0005176948450394379 -> xyz=-0.08171623350951565 0.3845030849366261 3.3590666332382993e-06 rpy=-1.5706673820173567 0.0015536598709241334 -0.0033016791726087685
- joint panda_joint6: origin xyz=-0.00012809341151093876 0.0006114705144863913 0.00038038616638708453 rpy=1.5678903763020455 0.0008804283250090152 0.0034804960271833806 -> xyz=-0.00011715350243528765 0.00043182234242505446 0.0005076215433290673 rpy=1.5678257347531421 0.00011154392567364391 0.0015543224619519137
- joint panda_joint7: origin xyz=0.08519872598122621 4.308755776248788e-06 -0.0006108393557751972 rpy=1.5709914845994533 5.0372969287365315e-08 -0.0008706911908268 -> xyz=0.08777435808196205 3.654336215268937e-07 -0.0004295228322241959 rpy=1.570880084703017 5.259780031068042e-09 -0.00010721814207152154

File: urdf/gen3lite.urdf (robot description, URDF)
Before this commit: robot kinova, 16 links, 15 joints
Joints:
- joint ball_joint: origin xyz=0.00038860649894460975 -0.0005822849938650045 0.180196205872143 rpy=0.0 0.0 0.0 -> xyz=0.0012427126494462678 -0.0014339702286163775 0.18526544228489414 rpy=0.0 0.0 0.0

File: urdf/iiwa14.urdf (robot description, URDF)
Before this commit: robot iiwa14, 11 links, 10 joints
Joints:
- joint ball_joint: origin xyz=0 0 0.04 rpy=0 0 0 -> xyz=-6.883092077759519e-05 -0.00018701061367410447 0.04081277546913972 rpy=0 0 0

File: urdf/panda.urdf (robot description, URDF)
Before this commit: robot panda, 14 links, 13 joints
Joints:
- joint ball_joint: origin xyz=7.773732033005863e-05 -4.214022515884392e-05 0.030128297908475325 rpy=0.0 0.0 0.0 -> xyz= 0 0 0.04 rpy=0.0 0.0 0.0
