Commit message: add result

File: calibrated_urdf/fr3/fr3.urdf (robot description, URDF)
Before this commit: robot fr3, 35 links, 34 joints
Links:
- link fr3_link0: geometry collision mesh filename=/home/haocheng/kinematics_calibration/meshes/fr3/link0.stl; visual mesh filename=/home/haocheng/kinematics_calibration/meshes/fr3/link0.dae
- link fr3_link1: geometry collision mesh filename=/home/haocheng/kinematics_calibration/meshes/fr3/link1.stl; visual mesh filename=/home/haocheng/kinematics_calibration/meshes/fr3/link1.dae
- link fr3_link2: geometry collision mesh filename=/home/haocheng/kinematics_calibration/meshes/fr3/link2.stl; visual mesh filename=/home/haocheng/kinematics_calibration/meshes/fr3/link2.dae
- link fr3_link3: geometry collision mesh filename=/home/haocheng/kinematics_calibration/meshes/fr3/link3.stl; visual mesh filename=/home/haocheng/kinematics_calibration/meshes/fr3/link3.dae
- link fr3_link4: geometry collision mesh filename=/home/haocheng/kinematics_calibration/meshes/fr3/link4.stl; visual mesh filename=/home/haocheng/kinematics_calibration/meshes/fr3/link4.dae
- link fr3_link5: geometry collision mesh filename=/home/haocheng/kinematics_calibration/meshes/fr3/link5.stl; visual mesh filename=/home/haocheng/kinematics_calibration/meshes/fr3/link5.dae
- link fr3_link6: geometry collision mesh filename=/home/haocheng/kinematics_calibration/meshes/fr3/link6.stl; visual mesh filename=/home/haocheng/kinematics_calibration/meshes/fr3/link6.dae
- link fr3_link7: geometry collision mesh filename=/home/haocheng/kinematics_calibration/meshes/fr3/link7.stl; visual mesh filename=/home/haocheng/kinematics_calibration/meshes/fr3/link7.dae
Joints:
- joint ball_joint: origin xyz=-0.0009532878100493034 -0.007076722219108235 0.03288695104519633 rpy=0.0 0.0 0.0 -> xyz=-0.0018201675662181923 -0.008005260162147827 0.03370209400757424 rpy=0.0 0.0 0.0
- joint fr3_joint1: origin xyz=-3.295701924808144e-17 5.2073447226205284e-17 0.33299999999999996 rpy=2.585694601074373e-18 4.63659574334812e-17 -3.9656478986234326e-17 -> xyz=0 0 0.333 rpy=0 0 0
- joint fr3_joint2: origin xyz=5.869418375711751e-05 0.0001939723832802431 -3.670194687854397e-17 rpy=-1.5690786772693188 0.00045848424635134237 4.904285936386038e-08 -> xyz=0 0 0 rpy=-1.570796326794897 0 0
- joint fr3_joint3: origin xyz=3.8744898039278656e-05 -0.31683866158059126 0.0001939678565617864 rpy=1.5699048387754349 -0.0025935094040345974 0.00044580105394580335 -> xyz=0 -0.316 0 rpy=1.570796326794897 0 0
- joint fr3_joint4: origin xyz=0.08262176815070747 0.0002584536661555798 0.0008393392257505757 rpy=1.5690063131693404 0.0013408186114178542 0.0025724036827010125 -> xyz=0.0825 0 0 rpy=1.570796326794897 0 0
- joint fr3_joint5: origin xyz=-0.08205109851416617 0.38479619963549055 -0.0002565304331815365 rpy=-1.5718586038590292 0.010858758956538534 -0.001098262999299868 -> xyz=-0.0825 0.384 0 rpy=-1.570796326794897 0 0
- joint fr3_joint6: origin xyz=0.0008128881964471342 0.0006330526730437588 0.0007970940777894692 rpy=1.5664572121896663 0.0014906755867315669 0.010859816375511585 -> xyz=0 0 0 rpy=1.570796326794897 0 0
- joint fr3_joint7: origin xyz=0.08748340010901132 8.579191546737077e-06 -0.0006189665361707107 rpy=1.5701463930952917 -9.204242284835627e-07 -0.0014445973965424642 -> xyz=0.088 0 0 rpy=1.570796326794897 0 0

File: urdf/fr3.urdf (robot description, URDF)
Before this commit: robot fr3, 35 links, 34 joints
Links:
- link fr3_link0: geometry collision mesh filename=/home/haocheng/kinematics_calibration/meshes/fr3/link0.stl; visual mesh filename=/home/haocheng/kinematics_calibration/meshes/fr3/link0.dae
- link fr3_link1: geometry collision mesh filename=/home/haocheng/kinematics_calibration/meshes/fr3/link1.stl; visual mesh filename=/home/haocheng/kinematics_calibration/meshes/fr3/link1.dae
- link fr3_link2: geometry collision mesh filename=/home/haocheng/kinematics_calibration/meshes/fr3/link2.stl; visual mesh filename=/home/haocheng/kinematics_calibration/meshes/fr3/link2.dae
- link fr3_link3: geometry collision mesh filename=/home/haocheng/kinematics_calibration/meshes/fr3/link3.stl; visual mesh filename=/home/haocheng/kinematics_calibration/meshes/fr3/link3.dae
- link fr3_link4: geometry collision mesh filename=/home/haocheng/kinematics_calibration/meshes/fr3/link4.stl; visual mesh filename=/home/haocheng/kinematics_calibration/meshes/fr3/link4.dae
- link fr3_link5: geometry collision mesh filename=/home/haocheng/kinematics_calibration/meshes/fr3/link5.stl; visual mesh filename=/home/haocheng/kinematics_calibration/meshes/fr3/link5.dae
- link fr3_link6: geometry collision mesh filename=/home/haocheng/kinematics_calibration/meshes/fr3/link6.stl; visual mesh filename=/home/haocheng/kinematics_calibration/meshes/fr3/link6.dae
- link fr3_link7: geometry collision mesh filename=/home/haocheng/kinematics_calibration/meshes/fr3/link7.stl; visual mesh filename=/home/haocheng/kinematics_calibration/meshes/fr3/link7.dae
