Commit message: udpate: add fr3 model

File: urdf/fr3.urdf (robot description, URDF)
Before this commit: robot fr3, 30 links, 29 joints
Links:
- added link ball_link; visual sphere radius=0.005
- added link fr3_hand; visual mesh filename=../meshes/fr3/hand.dae
- added link fr3_hand_tcp
- added link fr3_leftfinger; visual mesh filename=../meshes/fr3/finger.dae
- added link fr3_rightfinger; visual mesh filename=../meshes/fr3/finger.dae
Joints:
- added joint ball_joint: type fixed, parent fr3_hand_tcp, child ball_link, origin xyz=-0.0018201675662181923 -0.008005260162147827 0.03370209400757424 rpy=0.0 0.0 0.0
- added joint fr3_finger_joint1: type prismatic, parent fr3_hand, child fr3_leftfinger, origin xyz=0 0 0.0584 rpy=0 0 0, axis 0 1 0, limit lower=0.0 upper=0.04 effort=100 velocity=0.2
- added joint fr3_finger_joint2: type prismatic, parent fr3_hand, child fr3_rightfinger, origin xyz=0 0 0.0584 rpy=0 0 0, axis 0 -1 0, limit lower=0.0 upper=0.04 effort=100 velocity=0.2, mimic joint=fr3_finger_joint1
- added joint fr3_hand_joint: type fixed, parent fr3_link8, child fr3_hand, origin xyz=0 0 0 rpy=0 0 -0.7853981633974483
- added joint fr3_hand_tcp_joint: type fixed, parent fr3_hand, child fr3_hand_tcp, origin xyz=0 0 0.1034 rpy=0 0 0
