Commit message: update

File: calibrated_urdf/fr3_1/fr3.urdf (robot description, URDF)
Before this commit: robot fr3, 35 links, 34 joints
Joints:
- joint ball_joint: origin xyz=-0.0009147108639550119 -1.7543200838832017e-05 0.035163972429055744 rpy=0.0 0.0 0.0 -> xyz=-0.0009147185555085236 -1.754088059546966e-05 0.03219708441643505 rpy=0.0 0.0 0.0
- joint fr3_joint1: origin xyz=9.503297615097784e-18 3.0897841913570455e-17 0.3330000000000001 rpy=5.231263930585714e-17 7.14396133978129e-17 -1.0136231261311921e-16 -> xyz=-2.447164727006978e-17 1.9977949979524458e-17 0.33299999999999996 rpy=-6.244163137498879e-19 5.291241641851583e-17 -7.58916466465139e-18
- joint fr3_joint2: origin xyz=0.00011848406791370634 0.0007721351341233517 5.33927965425088e-17 rpy=-1.5715949066072126 0.002709766529478309 4.667417361437788e-09 -> xyz=0.00011848018876511169 0.0007721360704577187 -3.2906633262855086e-17 rpy=-1.5715949103692501 0.0027097748375854397 1.3564567549358015e-09
- joint fr3_joint3: origin xyz=0.0004143533550402461 -0.31636787758969176 0.000772134673123417 rpy=1.5667768037147476 0.0008469782559060354 0.0025788418515213366 -> xyz=0.0004143611025519952 -0.3163679192395694 0.0007721355694101926 rpy=1.5667768015480488 0.0008469864213074005 0.0025788501485276023
- joint fr3_joint4: origin xyz=0.0824989016520337 7.698968541204212e-05 0.00037205071646055757 rpy=1.5702490139713587 0.0013331688648600686 -0.0008429699651316111 -> xyz=0.08249892692930846 7.69953320542652e-05 0.0003720962457431666 rpy=1.5702490139085936 0.0013331784547376676 -0.0008429759428888274
- joint fr3_joint5: origin xyz=-0.08243686955595247 0.3843324784646275 -7.680932297334456e-05 rpy=-1.5721498649391061 -0.00014291994039891394 -0.0012819815944365995 -> xyz=-0.08243687230014404 0.3843325184097344 -7.681242314871467e-05 rpy=-1.5721498726877208 -0.00014290889534403448 -0.0012819758064718696
- joint fr3_joint6: origin xyz=-0.00012939884182346838 0.0004303391361667452 0.00033267166420328557 rpy=1.563510263736694 -0.00021449403094109997 -0.00014116800479009467 -> xyz=-0.00012940369565664272 0.0004303357531086777 0.00033271010713557814 rpy=1.5635102601005593 -0.00021718181070043167 -0.0001411606680153823
- joint fr3_joint7: origin xyz=0.08896198418934921 -1.5940331047446983e-05 -0.0004278812053006826 rpy=1.5708619226398732 1.2938894315897623e-07 0.00021486341430074264 -> xyz=0.08896136814223617 1.6872028485708933e-05 -0.00042788009467542104 rpy=1.5708619426031787 1.3974772537519443e-07 0.00021471961749753638
- joint fr3_joint8: origin xyz=0 0 0.107 rpy=0 0 0 -> xyz=0 0 0.110 rpy=0 0 0

File: urdf/fr3.urdf (robot description, URDF)
Before this commit: robot fr3, 35 links, 34 joints
Joints:
- joint fr3_joint8: origin xyz=0 0 0.107 rpy=0 0 0 -> xyz=0 0 0.110 rpy=0 0 0
